File: electronics/ESP-BOY-V1/ESP-BOY.kicad_sch (KiCad schematic)
At the start: 39 parts, among them J1 V_IN_TP, J10 USB_C_Receptacle, J2 3v3_TP, J3 TX_TP, J4 RX_TP, J5 DISP_BL_TP, J6 GND_A_TP, J7 GND_B_TP, J8 Micro_SD_Card, J9 Conn_01x08_Male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

Commit message: first routing pass
Parts:
- Q1: footprint Package_TO_SOT_THT:TO-92_Inline -> Package_TO_SOT_SMD:SOT-23
Changed lines of the file:
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@@
       (effects (font (size 1.27 1.27)) (justify left))
     )
-    (property "Footprint" "Package_TO_SOT_THT:TO-92_Inline" (id 2) (at 140.462 111.887 0)
+    (property "Footprint" "Package_TO_SOT_SMD:SOT-23" (id 2) (at 140.462 111.887 0)
       (effects (font (size 1.27 1.27) italic) (justify left) hide)
     )
@@
     )
     (path "/d4e58911-9ef0-4855-bb10-bf00f0c3ae7f"
-      (reference "Q1") (unit 1) (value "2N3904") (footprint "Package_TO_SOT_THT:TO-92_Inline")
+      (reference "Q1") (unit 1) (value "2N3904") (footprint "Package_TO_SOT_SMD:SOT-23")
     )
     (path "/28aefc84-1f0c-415b-b337-ae32b0353648"

Commit message: did more pcb layout stuff
Parts:
- added C8, C9: 22pF, Capacitor_SMD:C_0805_2012Metric, symbol Device:C
- added D1, D2: LED, LED_SMD:LED_1206_3216Metric, symbol Device:LED
- added R7, R8: R, Resistor_SMD:R_0805_2012Metric, symbol Device:R
Connections:
- net +3V3: now also C8.1, C9.1, D1.2 (A)
- net +5V: now also C6.1, C7.1, SW1.2 (B), U2.3 (VI), D2.2 (A)
- net GND: now also C8.2, C9.2, R7.2, R8.2
- net V_IN: no longer C6.1, C7.1
- new net: D2.1 (K), R8.1
- new net: D1.1 (K), R7.1
