File: electronics/ESP-BOY-V1/ESP-BOY.kicad_pcb (KiCad board)
At the start: 2 copper layers, 100.9 x 47.2 mm, 39 parts, among them J1 V_IN_TP, J10 USB_C_Receptacle, J2 3v3_TP, J3 TX_TP, J4 RX_TP, J5 DISP_BL_TP, J6 GND_A_TP, J7 GND_B_TP, J8 Micro_SD_Card, J9 Conn_01x08_Male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

Commit message: first routing pass
Parts:
- moved J7 81.6 mm to (143.5, 109.2)
- moved J1 77.8 mm to (143.6, 103.8)
- moved J2 65.4 mm to (118.9, 124.2)
- moved J4 47.4 mm to (117.5, 112.5)
- moved J8 44.6 mm to (98.8, 126.6), turned to 0 degrees
- moved J3 43.7 mm to (119.9, 116.7)
- moved J6 38.1 mm to (118.9, 129.3)
- moved SW10 28.3 mm to (60.8, 89.8), turned to 180 degrees
- moved J5 25.6 mm to (83.7, 118.7)
- moved SW4 23.1 mm to (61.0, 93.5), turned to 180 degrees
- moved SW9 14.4 mm to (89.2, 127.6)
- moved J10 8.02 mm to (127.0, 90.8)
- moved J9 7.84 mm to (76.7, 96.3)
- moved SW8 6.11 mm to (64.4, 109.1)
- moved U3 6.07 mm to (98.9, 103.4)
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Routing:
- net LEFT_BUTTON: track 0.00 -> 58.2 mm, vias 0 -> 1
- net ESP_PROG: track 0.00 -> 54.2 mm, vias 0 -> 1
- net DOWN_BUTTON: track 0.00 -> 48.7 mm, vias 0 -> 1
- net RIGHT_BUTTON: track 0.00 -> 48.6 mm, vias 0 -> 1
- net UP_BUTTON: track 0.00 -> 48.5 mm, vias 0 -> 1
- net ESP_EN: track 0.00 -> 48.2 mm, vias 0 -> 1
- net GND: track 0.00 -> 45.1 mm, vias 0 -> 28
- net DISP_CS: track 0.00 -> 42.9 mm, vias 0 -> 1
- net USB_TX: track 0.00 -> 41.6 mm, vias 0 -> 3
- net USB_RX: track 0.00 -> 40.5 mm, vias 0 -> 2
- net START_BUTTON: track 0.00 -> 38.6 mm, vias 0 -> 1
- net DISP_MOSI: track 0.00 -> 35.1 mm, vias 0 -> 2
- net DISP_CLK: track 0.00 -> 34.9 mm, vias 0 -> 3
- net A_BUTTON: track 0.00 -> 33.0 mm, vias 0 -> 1
- net DISP_RST: track 0.00 -> 31.0 mm, vias 0 -> 3
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- added copper zone on In2.Cu, net +3V3
- added copper zone on B.Cu, net GND
- added copper zone on F.Cu, net GND
- added copper zone on In1.Cu, net GND
Other:
- board size 100.9 x 47.2 mm -> 101.6 x 47.8 mm
- copper layers 2 -> 4

Commit message: did more pcb layout stuff
Parts:
- added C8: 22pF, Capacitor_SMD:C_0805_2012Metric, B.Cu at (111.8, 96.9)
- added C9: 22pF, Capacitor_SMD:C_0805_2012Metric, B.Cu at (111.8, 99.1)
- added D1: LED, LED_SMD:LED_1206_3216Metric, F.Cu at (138.0, 96.6)
- added D2: LED, LED_SMD:LED_1206_3216Metric, F.Cu at (138.0, 94.1)
- added R7: R, Resistor_SMD:R_0805_2012Metric, B.Cu at (137.6, 96.5)
- added R8: R, Resistor_SMD:R_0805_2012Metric, B.Cu at (137.5, 94.2)
- moved J7 9.49 mm to (145.5, 99.9)
- moved J3 6.71 mm to (114.6, 112.6)
- moved J1 5.21 mm to (140.1, 99.9)
- moved R5 3.14 mm to (133.7, 99.0)
- moved R6 3.14 mm to (131.7, 99.0)
- moved J4 0.77 mm to (118.2, 112.6)
- turned C1 to 180 degrees
- turned C3 to 180 degrees
Connections:
- C6 pad 1: V_IN -> +5V
- C7 pad 1: V_IN -> +5V
- SW1 pad 2: Net-(SW1-Pad2) -> +5V
- U2 pad 3: Net-(SW1-Pad2) -> +5V
Routing:
- net +5V: track 0.00 -> 54.8 mm, vias 0 -> 3
- net V_IN: track 2.16 -> 27.2 mm
- net GND: track 45.1 -> 22.3 mm, vias 28 -> 49
- net +3V3: track 18.1 -> 29.8 mm, vias 9 -> 11
- net USB_TX: track 41.6 -> 51.1 mm
- net Net-(J10-PadA5): track 0.00 -> 8.49 mm, vias 0 -> 2
- net Net-(J10-PadA4): track 2.66 -> 9.94 mm
- net USB_RX: track 40.5 -> 47.0 mm
- net Net-(D1-Pad1): track 0.00 -> 3.10 mm, vias 0 -> 1
- net Net-(D2-Pad1): track 0.00 -> 3.05 mm, vias 0 -> 1
- net Net-(C1-Pad1): track 12.6 -> 11.0 mm
- net Net-(C3-Pad1): track 12.1 -> 10.7 mm
- net DISP_MOSI: track 35.1 -> 33.9 mm
- net B_BUTTON: track 28.6 -> 29.5 mm
- net ESP_PROG: track 54.2 -> 54.9 mm
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
Commit message: remove bt stuff
Parts:
- moved D1 5.21 mm to (138.0, 91.4)
- moved R7 5.21 mm to (137.6, 91.3)
Routing:
- net +5V: track 54.8 -> 26.4 mm, vias 3 -> 6
- net +3V3: track 29.8 -> 32.9 mm
- added copper zone on In2.Cu, net +5V
